File: Schematics/SonicDuino/sonicduino/sonicduino.sch (KiCad schematic (older format))
At the start: 8 parts, among them J1 Conn_01x06_Male, J2 Conn_01x08_Male, J3 Conn_01x06_Male, U1 ATmega328P-PU, Y1 16 MHz Crystal

Commit message: Complete initial version of SonicDuino schematic
Parts:
- added D?: LED, symbol Device:LED
- added J4: Conn_01x05_Male, symbol Connector:Conn_01x05_Male
- added J4: Conn_01x06_Male, symbol Connector:Conn_01x06_Male
- added R2: 1k, symbol Device:R_US
Connections:
- net at U1.15 (PB1): now also J4.1 (Pin_1)
- net at U1.16 (PB2): now also J4.2 (Pin_2)
- net at J1.3 (Pin_3), U1.17 (PB3): now also J4.3 (Pin_3)
- net at J1.2 (Pin_2), U1.18 (PB4): now also J4.4 (Pin_4)
- net at J1.1 (Pin_1), U1.19 (PB5): now also J4.5 (Pin_5), R2.1
- net at C1.1, C2.1, J1.5 (Pin_5)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: now also D?.1 (K)
- net at U1.23 (PC0): now also J4.1 (Pin_1)
- net at U1.24 (PC1): now also J4.2 (Pin_2)
- net at U1.25 (PC2): now also J4.3 (Pin_3)
- net at U1.26 (PC3): now also J4.4 (Pin_4)
- net at U1.27 (PC4): now also J4.5 (Pin_5)
- net at U1.28 (PC5): now also J4.6 (Pin_6)
- new net: D?.2 (A), R2.2
Other:
- moved on the sheet: J2, J3
Changed lines of the file:
@@
 EESchema Schematic File Version 4
-EELAYER 30 0
+LIBS:sonicduino-cache
+EELAYER 29 0
 EELAYER END
 $Descr A4 11693 8268
@@
 U 1 1 5DF6AAEE
 P 5400 3850
-F 0 "U1" H 4800 3950 50  0000 R CNN
-F 1 "ATmega328P-PU" V 4756 3805 50  0000 R CNN
+F 0 "U1" H 5450 4150 50  0000 R CNN
+F 1 "ATmega328P-PU" V 5350 3950 50  0000 R CNN
 F 2 "Package_DIP:DIP-28_W7.62mm" H 5400 3850 50  0001 C CIN
 F 3 "http://ww1.microchip.com/downloads/en/DeviceDoc/ATmega328_P%20AVR%20MCU%20with%20picoPower%20Technology%20Data%20Sheet%2040001984A.pdf" H 5400 3850 50  0001 C CNN
@@
 Connection ~ 3650 5450
 Wire Wire Line
-	3650 5450 5400 5450
+	3650 5450 4600 5450
 Wire Wire Line
 	3250 5450 3650 5450
@@
 	3900 3550 3900 1800
 Wire Wire Line
-	3900 1800 6300 1800
-Wire Wire Line
-	6300 1800 6300 3150
+	3900 1800 4600 1800
+Wire Wire Line
+	6300 1800 6300 2450
 Wire Wire Line
 	6300 3150 6000 3150
@@
 L Connector:Conn_01x08_Male J2
 U 1 1 5DF864DC
-P 6950 4450
-F 0 "J2" H 7100 4900 50  0000 R CNN
-F 1 "Conn_01x08_Male" H 7300 4900 50  0001 R CNN
-F 2 "" H 6950 4450 50  0001 C CNN
-F 3 "~" H 6950 4450 50  0001 C CNN
-	1    6950 4450
+P 7900 4450
+F 0 "J2" H 7800 4450 50  0000 R CNN
+F 1 "Conn_01x08_Male" H 8250 4900 50  0001 R CNN
+F 2 "" H 7900 4450 50  0001 C CNN
+F 3 "~" H 7900 4450 50  0001 C CNN
+	1    7900 4450
 	-1   0    0    -1
 $EndComp
 Wire Wire Line
-	6750 4150 6100 4150
+	7700 4150 6100 4150
 Connection ~ 6100 4150
 Wire Wire Line
-	6750 4250 6350 4250
+	7700 4250 6350 4250
 Wire Wire Line
 	6350 4250 6350 4350
@@
 	6350 4350 6000 4350
 Wire Wire Line
-	6750 4350 6400 4350
+	7700 4350 6400 4350
 Wire Wire Line
 	6400 4350 6400 4450
@@
 	6400 4450 6000 4450
 Wire Wire Line
-	6750 4450 6450 4450
+	7700 4450 6450 4450
 Wire Wire Line
 	6450 4550 6000 4550
 Wire Wire Line
-	6750 4550 6500 4550
+	7700 4550 6500 4550
 Wire Wire Line
 	6500 4550 6500 4650
@@
 	6500 4650 6000 4650
 Wire Wire Line
-	6750 4650 6550 4650
+	7700 4650 6550 4650
 Wire Wire Line
 	6550 4650 6550 4750
@@
 	6550 4750 6000 4750
 Wire Wire Line
-	6750 4850 6750 5450
-Wire Wire Line
-	6750 5450 5400 5450
-Connection ~ 5400 5450
-Wire Wire Line
-	6750 4750 6650 4750
+	7700 4750 6650 4750
 Wire Wire Line
 	4300 5650 6100 5650
@@
 L Connector:Conn_01x06_Male J3
 U 1 1 5DFA551A
-P 7200 3300
-F 0 "J3" H 7350 3650 50  0000 R CNN
-F 1 "Conn_01x06_Male" H 7550 2800 50  0001 R CNN
-F 2 "" H 7200 3300 50  0001 C CNN
-F 3 "~" H 7200 3300 50  0001 C CNN
-	1    7200 3300
+P 7900 3150
+F 0 "J3" H 7800 3150 50  0000 R CNN
+F 1 "Conn_01x06_Male" H 8250 2650 50  0001 R CNN
+F 2 "" H 7900 3150 50  0001 C CNN
+F 3 "~" H 7900 3150 50  0001 C CNN
+	1    7900 3150
 	-1   0    0    -1
 $EndComp
 Wire Wire Line
-	7000 3100 6450 3100
-Wire Wire Line
-	6450 3100 6450 3250
+	7700 2950 6900 2950
+Wire Wire Line
+	6900 2950 6450 3250
 Wire Wire Line
 	6450 3250 6300 3250
 Connection ~ 6300 3250
 Wire Wire Line
-	7000 3200 6600 3200
-Wire Wire Line
-	6600 3200 6600 3350
-Wire Wire Line
-	6600 3350 6200 3350
+	7700 3050 6900 3050
+Wire Wire Line
+	6900 3050 6500 3350
+Wire Wire Line
+	6500 3350 6200 3350
 Connection ~ 6200 3350
 Wire Wire Line
@@
 	6600 3400 6700 3400
 Wire Wire Line
-	6700 3400 6700 3300
-Wire Wire Line
-	6700 3300 7000 3300
-Wire Wire Line
-	7000 3400 6750 3400
-Wire Wire Line
-	6750 3400 6750 3900
-Wire Wire Line
-	6750 3900 7100 3900
-Wire Wire Line
-	7100 3900 7100 4950
+	6700 3400 6700 3150
+Wire Wire Line
+	6700 3150 7700 3150
+Wire Wire Line
+	7700 3250 6750 3250
+Wire Wire Line
+	6750 3250 6750 4050
+Wire Wire Line
+	6750 4050 7100 4050
+Wire Wire Line
+	7100 4050 7100 4950
 Wire Wire Line
 	7100 4950 6000 4950
 Wire Wire Line
-	7000 3500 6850 3500
-Wire Wire Line
-	6850 3500 6850 3800
-Wire Wire Line
-	6850 3800 7200 3800
-Wire Wire Line
-	7200 3800 7200 5050
+	7700 3350 6850 3350
+Wire Wire Line
+	6850 3350 6850 4000
+Wire Wire Line
+	6850 4000 7200 4000
+Wire Wire Line
+	7200 4000 7200 5050
 Wire Wire Line
 	7200 5050 6000 5050
@@
 	6000 2650 6950 2650
 Wire Wire Line
-	6950 2650 6950 3600
-Wire Wire Line
-	6950 3600 7000 3600
+	6950 2650 6950 3450
+Wire Wire Line
+	6950 3450 7700 3450
+$Comp
+L Connector:Conn_01x05_Male J4
+U 1 1 5DF78071
+P 7900 2250
+F 0 "J4" H 7872 2228 50  0000 R CNN
+F 1 "Conn_01x05_Male" H 7872 2183 50  0001 R CNN
+F 2 "" H 7900 2250 50  0001 C CNN
+F 3 "~" H 7900 2250 50  0001 C CNN
+	1    7900 2250
+	-1   0    0    -1
+$EndComp
+Wire Wire Line
+	7700 2050 6400 2050
+Wire Wire Line
+	6400 2050 6400 2750
+Wire Wire Line
+	6400 2750 6000 2750
+Wire Wire Line
+	7700 2150 6500 2150
+Wire Wire Line
+	6500 2150 6500 2850
+Wire Wire Line
+	6500 2850 6000 2850
+Wire Wire Line
+	7700 2250 6600 2250
+Wire Wire Line
+	6600 2250 6600 2950
+Wire Wire Line
+	6600 2950 6100 2950
+Connection ~ 6100 2950
+Wire Wire Line
+	7700 2350 6700 2350
+Wire Wire Line
+	6700 2350 6700 3050
+Wire Wire Line
+	6700 3050 6200 3050
+Connection ~ 6200 3050
+Wire Wire Line
+	7700 2450 6300 2450
+Connection ~ 6300 2450
+Wire Wire Line
+	6300 2450 6300 3150
+$Comp
+L Device:LED D?
+U 1 1 5DF87E1C
+P 4600 4500
+F 0 "D?" V 4639 4383 50  0001 R CNN
+F 1 "LED" V 4593 4383 50  0000 R CNN
+F 2 "" H 4600 4500 50  0001 C CNN
+F 3 "~" H 4600 4500 50  0001 C CNN
+	1    4600 4500
+	0    -1   -1   0
+$EndComp
+$Comp
+L Device:R_US R2
+U 1 1 5DF8918B
+P 4600 3850
+F 0 "R2" H 4668 3896 50  0000 L CNN
+F 1 "1k" H 4668 3805 50  0000 L CNN
+F 2 "" V 4640 3840 50  0001 C CNN
+F 3 "~" H 4600 3850 50  0001 C CNN
+	1    4600 3850
+	1    0    0    -1
+$EndComp
+Wire Wire Line
+	4600 4000 4600 4350
+Wire Wire Line
+	4600 4650 4600 5450
+Connection ~ 4600 5450
+Wire Wire Line
+	4600 5450 5400 5450
+Wire Wire Line
+	4600 3700 4600 1800
+Connection ~ 4600 1800
+Wire Wire Line
+	4600 1800 6300 1800
+$Comp
+L Connector:Conn_01x06_Male J4
+U 1 1 5DF93A6C
+P 7900 3750
+F 0 "J4" H 7800 3750 50  0000 R CNN
+F 1 "Conn_01x06_Male" H 8250 3250 50  0001 R CNN
+F 2 "" H 7900 3750 50  0001 C CNN
+F 3 "~" H 7900 3750 50  0001 C CNN
+	1    7900 3750
+	-1   0    0    -1
+$EndComp
+Wire Wire Line
+	7700 3550 7450 3550
+Wire Wire Line
+	7450 3550 7450 3650
+Wire Wire Line
+	7450 3650 6450 3650
+Wire Wire Line
+	6450 3650 6450 3550
+Wire Wire Line
+	6450 3550 6000 3550
+Wire Wire Line
+	7550 3650 7550 3700
+Wire Wire Line
+	7550 3700 6350 3700
+Wire Wire Line
+	6350 3700 6350 3650
+Wire Wire Line
+	6350 3650 6000 3650
+Wire Wire Line
+	7550 3650 7700 3650
+Wire Wire Line
+	6000 3750 7700 3750
+Wire Wire Line
+	6000 3850 7700 3850
+Wire Wire Line
+	7700 3950 6000 3950
+Wire Wire Line
+	7250 4050 7250 4100
+Wire Wire Line
+	7250 4100 6350 4100
+Wire Wire Line
+	6350 4100 6350 4050
+Wire Wire Line
+	6350 4050 6000 4050
+Wire Wire Line
+	7250 4050 7700 4050
+Wire Wire Line
+	7700 4850 7700 5450
+Wire Wire Line
+	7700 5450 5400 5450
+Connection ~ 5400 5450
 $EndSCHEMATC
