File: Schematics/PowerSupply/powersupply/powersupply.kicad_pcb (KiCad board)
At the start: 2 copper layers, 12 parts, among them J1 +/- 15V Regulated, J2 +/- 18V unregulated, J3 Transformer Secondary, U1 L7815, U2 L7915

Commit message: Add final version of the powersupply pcb
Parts:
- C1, C2: footprint Capacitor_THT:CP_Radial_D10.0mm_P5.00mm -> Capacitor_THT:CP_Radial_D17.0mm_P7.50mm
- C3, C4, C5, C6: footprint Capacitor_THT:C_Rect_L4.0mm_W2.5mm_P2.50mm -> Capacitor_THT:C_Rect_L9.0mm_W2.5mm_P7.50mm_MKT
- moved D1 7.44 mm to (104.1, 114.8)
- moved J3 5.41 mm to (124.2, 111.8)
- moved C1 3.84 mm to (142.7, 120.3)
- moved C4 2.89 mm to (154.9, 99.4)
- moved C3 2.68 mm to (154.7, 116.3)
- moved C2 1.55 mm to (142.5, 100.7)
Routing:
- net Net-(C2-Pad2): track 108.5 -> 122.4 mm
- net Net-(C1-Pad1): track 119.6 -> 131.4 mm
- net Net-(D1-Pad3): track 18.2 -> 20.7 mm
- net Net-(D1-Pad2): track 18.4 -> 20.4 mm
