File: Schematics/Amplifier/Amplifier2.sch (KiCad schematic (older format))
At the start: 54 parts, among them J1 Conn_01x03_Female, J2 Conn_01x03_Female, J3 Conn_01x03_Female, J4 Conn_01x03_Female, Q1 BD139, Q2 BD138, Q3 BC556, Q4 BC546, Q5 BC556, Q6 BC546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

Commit message: Modify the amp schematic
Parts:
- removed C8: 1000u, Capacitor_THT:C_Radial_D16.0mm_H25.0mm_P7.50mm, symbol Device:CP
- removed Q5: BC556, Package_TO_SOT_THT:TO-92_Inline, symbol Transistor_BJT:BC556
- removed Q6: BC546, Package_TO_SOT_THT:TO-92_Inline, symbol Transistor_BJT:BC546
- removed R13, R16: 15k, Resistor_THT:R_Axial_DIN0204_L3.6mm_D1.6mm_P7.62mm_Horizontal, symbol Device:R
- removed R14, R15: 220k, Resistor_THT:R_Axial_DIN0204_L3.6mm_D1.6mm_P7.62mm_Horizontal, symbol Device:R
- removed R17, R18, R19, R22: 220, Resistor_THT:R_Axial_DIN0204_L3.6mm_D1.6mm_P7.62mm_Horizontal, symbol Device:R
- removed R20, R21: 4k7, Resistor_THT:R_Axial_DIN0204_L3.6mm_D1.6mm_P7.62mm_Horizontal, symbol Device:R
- removed R23, R24: 0.22, Resistor_THT:R_Axial_Power_L20.0mm_W6.4mm_P22.40mm, symbol Device:R
- added D5, D6, D7, D8: 1N4001, Diode_THT:D_DO-41_SOD81_P10.16mm_Horizontal, symbol Diode:1N4001
- added Q5: BC546, Package_TO_SOT_THT:TO-92_Inline, symbol Transistor_BJT:BC546
- added Q6: BC556, Package_TO_SOT_THT:TO-92_Inline, symbol Transistor_BJT:BC556
- R11, R8: value 220k -> 0.22; footprint Resistor_THT:R_Axial_DIN0204_L3.6mm_D1.6mm_P7.62mm_Horizontal -> Resistor_THT:R_Axial_Power_L20.0mm_W6.4mm_P22.40mm
- R12, R7: value 15k -> 10k
- R5, R6: value 4k7 -> 10k
Connections:
- net at C12.1, J4.1 (Pin_1), Q1.2 (C)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: now also Q4.1 (C), R5.1, R6.1, Q5.1 (C); no longer R7.1
- net at D1.2 (A), R5.2: now also C3.1, Q4.2 (B); no longer Q1.3 (B)
- net at C9.2, J4.2 (Pin_2), Q2.2 (C)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: now also Q3.1 (C), R7.2, Q6.1 (C)
- net at R6.2: now also C5.1, D5.2 (A), Q5.2 (B); no longer Q4.1 (C)
- net at C4.2, R12.1: now also D4.1 (K), Q3.2 (B); no longer Q4.2 (B), R11.2
- net at J3.3 (Pin_3): now also R11.1, R8.2
- net at Q4.3 (E): now also Q1.3 (B)
- net at Q3.3 (E): now also Q2.3 (B)
- net at Q8.1 (E): now also R11.2
- net at Q7.1 (E): now also R8.1
- net at Q8.3 (B): now also Q6.3 (E); no longer D4.1 (K)
- net at D3.2 (A): now also D2.1 (K); no longer Q7.3 (B)
- net at C6.2: now also R7.1, D8.1 (K), Q6.2 (B)
- new net: C7.1, R10.1, R9.2
- new net: D1.1 (K), D2.2 (A)
- new net: D5.1 (K), D6.2 (A)
- new net: D6.1 (K), D7.2 (A)
- new net: Q5.3 (E), Q7.3 (B)
- new net: D7.1 (K), D8.2 (A)
Other:
- moved on the sheet: C3, C4, C7, C9, D1, D2, Q1, Q2, Q3, Q4, R10, R9
